Commit message: Improve dual-lidar mission behavior and world simulation tuning

File: src/ridgeback_vision_detection/urdf/camera_extras.urdf.xacro (robot description, xacro)
@@ -1,27 +1,25 @@
 <?xml version="1.0"?>
 <robot xmlns:xacro="http://ros.org/wiki/xacro">
-  <link name="camera_extra_link">
+  <link name="d455_link">
     <visual>
-      <geometry><box size="0.1 0.1 0.1"/></geometry>
-      <material name="yellow"/>
+      <geometry><box size="0.124 0.029 0.026"/></geometry>
+      <material name="black"/>
     </visual>
     <collision>
-      <geometry><box size="0.1 0.1 0.1"/></geometry>
+      <geometry><box size="0.124 0.029 0.026"/></geometry>
     </collision>
     <inertial>
-      <mass value="0.1"/>
+      <mass value="0.072"/>
       <origin xyz="0 0 0" rpy="0 0 0"/>
-      <inertia ixx="0.000166" ixy="0" ixz="0" iyy="0.000166" iyz="0" izz="0.000166"/>
+      <inertia ixx="2e-5" ixy="0" ixz="0" iyy="2e-5" iyz="0" izz="2e-5"/>
     </inertial>
   </link>
-  <joint name="camera_extra_joint" type="revolute">
+  <joint name="d455_joint" type="fixed">
     <parent link="chassis_link"/>
-    <child link="camera_extra_link"/>
-    <origin xyz="0.6 0 0.8" rpy="0 0.15 0"/>
-    <axis xyz="0 1 0"/>
-    <limit lower="0" upper="0" effort="0" velocity="0"/>
+    <child link="d455_link"/>
+    <origin xyz="0.0 0 0.8" rpy="0 0 0"/>
   </joint>
-  <gazebo reference="camera_extra_link">
-    <sensor name="camera_sensor" type="camera">
+  <gazebo reference="d455_link">
+    <sensor name="d455_sensor" type="camera">
       <camera>
         <horizontal_fov>1.047</horizontal_fov>
@@ -39,7 +37,7 @@
       <update_rate>10</update_rate>
       <visualize>true</visualize>
-      <topic>/camera_sensor/image_raw</topic>
-      <gz_frame_id>camera_extra_link</gz_frame_id>
-      <ignition_frame_id>camera_extra_link</ignition_frame_id>
+      <topic>/camera_d455/image_raw</topic>
+      <gz_frame_id>d455_link</gz_frame_id>
+      <ignition_frame_id>d455_link</ignition_frame_id>
     </sensor>
   </gazebo>

File: src/ridgeback_vision_detection/urdf/lidar_extras.urdf.xacro (robot description, xacro)
@@ -1,5 +1,5 @@
 <?xml version="1.0"?>
 <robot xmlns:xacro="http://ros.org/wiki/xacro">
-  <link name="lidar_link">
+  <link name="lidar_front_link">
     <visual>
       <geometry><cylinder radius="0.05" length="0.07"/></geometry>
@@ -15,21 +15,61 @@
     </inertial>
   </link>
-  <joint name="lidar_joint" type="fixed">
+  <joint name="lidar_front_joint" type="fixed">
     <parent link="chassis_link"/>
-    <child link="lidar_link"/>
+    <child link="lidar_front_link"/>
     <origin xyz="0.35 0.0 0.32" rpy="0 0 0"/>
   </joint>
-  <gazebo reference="lidar_link">
-    <sensor name="lidar" type="gpu_lidar">
+  <link name="lidar_rear_link">
+    <visual>
+      <geometry><cylinder radius="0.05" length="0.07"/></geometry>
+      <material name="black"/>
+    </visual>
+    <collision>
+      <geometry><cylinder radius="0.05" length="0.07"/></geometry>
+    </collision>
+    <inertial>
+      <mass value="0.2"/>
+      <origin xyz="0 0 0" rpy="0 0 0"/>
+      <inertia ixx="1e-4" ixy="0" ixz="0" iyy="1e-4" iyz="0" izz="1e-4"/>
+    </inertial>
+  </link>
+  <joint name="lidar_rear_joint" type="fixed">
+    <parent link="chassis_link"/>
+    <child link="lidar_rear_link"/>
+    <origin xyz="-0.35 0.0 0.32" rpy="0 0 3.14159"/>
+  </joint>
+  <gazebo reference="lidar_front_link">
+    <sensor name="lidar_front" type="gpu_lidar">
       <update_rate>10</update_rate>
       <topic>scan</topic>
-      <gz_frame_id>lidar_link</gz_frame_id>
-      <ignition_frame_id>lidar_link</ignition_frame_id>
+      <gz_frame_id>lidar_front_link</gz_frame_id>
+      <ignition_frame_id>lidar_front_link</ignition_frame_id>
       <ray>
         <scan>
           <horizontal>
             <samples>720</samples>
-            <min_angle>-3.14159</min_angle>
-            <max_angle>3.14159</max_angle>
+            <min_angle>-2.35619</min_angle>
+            <max_angle>2.35619</max_angle>
+          </horizontal>
+        </scan>
+        <range>
+          <min>0.12</min>
+          <max>12.0</max>
+        </range>
+      </ray>
+    </sensor>
+  </gazebo>
+  <gazebo reference="lidar_rear_link">
+    <sensor name="lidar_rear" type="gpu_lidar">
+      <update_rate>10</update_rate>
+      <topic>scan_rear</topic>
+      <gz_frame_id>lidar_rear_link</gz_frame_id>
+      <ignition_frame_id>lidar_rear_link</ignition_frame_id>
+      <ray>
+        <scan>
+          <horizontal>
+            <samples>720</samples>
+            <min_angle>-2.35619</min_angle>
+            <max_angle>2.35619</max_angle>
           </horizontal>
         </scan>
